File: ZXSpider48.kicad_pcb (KiCad board)
At the start: 2 copper layers, 213.5 x 130.5 mm, 151 parts, among them J1 Barrel_Jack_Switch, J11 EAR/MIC, J12 KB_CONN_05, J14 RESET, J15 ZX_48K_EDGE, J16 DB9_Pins, J17 ON/OFF, J18 JOYSTICK_ON_OFF, J19 AY3_IOB, J2 JTAG, J20 AY3_IOA, J3 9V, J4 AUDIO, J5 ROM_SW, J6 M-DIN KMDGX-9S-BS-1, J7 SPK_ON_OFF, J8 KB_CON_08, Q1 BC517, Q10 BC560, Q11 BC560, Q12 BC560, Q13 BC560, Q14 BC560, Q15 BC560, Q2 BC548, Q8 BC560, Q9 BC560, U1 AY-3-8912, U10 27C256, U11 74HCT240, U16 74LS138, U18 74LS00, U2 EPM7128SLC84-10, U3 LM7805_TO220, U4 AY-3-8910, U5 HM62256, U6 74HC04, U7 HM62256, U8 Z80, U9 74LS32, Y2 14.000 Mhz

Commit message: Add files via upload
Corrected R58 value 470R
Added jumper for EPROM/EEPROM select
Added jumper notations
Added more buffers to clock signal
Parts:
- added J9: UV/EEPROM, Connector_PinHeader_2.54mm:PinHeader_2x02_P2.54mm_Vertical, F.Cu at (122.2, 87.4)
- HBL1, HBR1, HTM1: footprint MountingHole:MountingHole_3.2mm_M3 -> _MOD:MountingHole_3.3mm Spectrum
- HLM1, HRM1: footprint MountingHole:MountingHole_5.3mm_M5 -> _MOD:MountingHole_5mm Spectrum
- J18: value JOYSTICK_ON_OFF -> JS_ENABLE
- R58: value 470K -> 470R
- U10: value 27C256 -> 27/28C256
- moved R74 83.6 mm to (111.7, 80.6)
- moved J5 80.6 mm to (115.0, 84.8), turned to 0 degrees
- moved Y2 27.4 mm to (100.9, 136.8)
- moved C20 17.3 mm to (93.3, 145.6), turned to 180 degrees
- moved R2 9.70 mm to (35.9, 50.0), turned to 0 degrees
- moved R3 9.67 mm to (36.0, 52.5), turned to 0 degrees
- moved R1 9.66 mm to (36.0, 47.5), turned to 0 degrees
- moved R50 8.20 mm to (88.0, 132.3)
- moved R54 7.64 mm to (79.8, 145.7), turned to 0 degrees
- moved R17 7.64 mm to (37.2, 36.1), turned to -90 degrees
- moved R15 7.59 mm to (30.2, 36.0), turned to -90 degrees
- moved R16 7.58 mm to (32.4, 36.0), turned to -90 degrees
- moved C5 4.49 mm to (99.2, 146.2), turned to 0 degrees
- moved J6 2.00 mm to (35.2, 29.4)
- moved J2 0.73 mm to (116.0, 142.7)
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Connections:
- R1 pad 1: Net-(J6-Pad7) -> Net-(D3-A)
- R15 pad 1: Net-(D3-A) -> Net-(J6-Pad7)
- R15 pad 2: Net-(J6-Pad7) -> Net-(D3-A)
- R16 pad 1: Net-(D4-A) -> Net-(J6-Pad3)
- R16 pad 2: Net-(J6-Pad3) -> Net-(D4-A)
- R17 pad 1: Net-(D5-A) -> Net-(J6-Pad1)
- R17 pad 2: Net-(J6-Pad1) -> Net-(D5-A)
- R2 pad 1: Net-(J6-Pad3) -> Net-(D4-A)
- R3 pad 1: Net-(J6-Pad1) -> Net-(D5-A)
- U10 pad 1: +5V -> Net-(J9-Pin_4)
- U10 pad 27: Net-(J5-Pin_2) -> Net-(J9-Pin_1)
- U6 pad 1: GND -> Net-(R50-Pad2)
- U6 pad 10: Net-(R54-Pad1) -> Net-(U6-Pad10)
- U6 pad 11: Net-(C20-Pad2) -> Net-(U6-Pad11)
- U6 pad 12: unconnected-(U6-Pad12) -> Net-(R54-Pad1)
- U6 pad 13: GND -> Net-(C20-Pad2)
- U6 pad 2: unconnected-(U6-Pad2) -> Net-(C20-Pad1)
- U6 pad 3: GND -> Net-(R54-Pad1)
- U6 pad 4: unconnected-(U6-Pad4) -> Net-(U6-Pad11)
- U6 pad 5: Net-(R50-Pad2) -> Net-(U6-Pad10)
- U6 pad 6: Net-(C20-Pad1) -> Net-(U6-Pad6)
- U6 pad 9: Net-(R54-Pad1) -> Net-(U6-Pad6)
Routing:
- net Net-(J5-Pin_2): track 108.0 -> 8.23 mm, vias 1 -> 0
- net GND: track 1020.8 -> 931.2 mm, vias 262 -> 266
- net Net-(J9-Pin_4): track 0.00 -> 22.4 mm, vias 0 -> 2
- net Net-(J6-Pad1): track 35.8 -> 16.8 mm
- net Net-(J6-Pad7): track 24.4 -> 6.21 mm
- net Net-(J9-Pin_1): track 0.00 -> 16.7 mm
- net Net-(J6-Pad3): track 31.0 -> 15.1 mm
- net Net-(R54-Pad1): track 16.2 -> 30.4 mm
- net +5V: track 975.2 -> 985.0 mm, vias 12 -> 14
- net Net-(C20-Pad2): track 15.5 -> 6.92 mm
- net Net-(J18-Pin_2): track 122.2 -> 114.3 mm
- net Net-(U6-Pad6): track 0.00 -> 7.62 mm
- net Net-(U6-Pad11): track 0.00 -> 7.62 mm
- net Net-(U6-Pad10): track 0.00 -> 7.62 mm
- net Net-(R50-Pad2): track 16.5 -> 9.12 mm
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Other:
- board text added: "1"
- board text added: "10"
- board text added: "2"
- board text added: "27/28C256"
- board text added: "3"
- board text added: "4"
- board text added: "9"
- board text added: "9V Out"
- board text added: "EEPROM 2-4/3-1 || EPROM 2-1/3-4 --"
- board text added: "Fit For +12V/-12V"
- board text added: "Hi/Lo"
- board text added: "JS_ENABLE"
- board text added: "JTAG"
- board text added: "ON/OFF"
- board text added: "RESET"
- board text added: "ROM SW"
- board text added: "SPK_Enable"
- board text added: "UVEPROM/EEPROM"
- board text removed: "27C256"
