File: ZXSpider48.kicad_pcb (KiCad board)
At the start: 2 copper layers, 213.5 x 130.5 mm, 152 parts, among them J1 Barrel_Jack_Switch, J11 EAR/MIC, J12 KB_CONN_05, J14 RESET, J15 ZX_48K_EDGE, J16 DB9_Pins, J17 ON/OFF, J18 JS_ENABLE, J19 AY3_IOB, J2 JTAG, J20 AY3_IOA, J3 9V, J4 AUDIO, J5 ROM_SW, J6 M-DIN KMDGX-9S-BS-1, J7 SPK_ON_OFF, J8 KB_CON_08, J9 UV/EEPROM, Q1 BC517, Q10 BC560, Q11 BC560, Q12 BC560, Q13 BC560, Q14 BC560, Q15 BC560, Q2 BC548, Q8 BC560, Q9 BC560, U1 AY-3-8912, U10 27/28C256, U11 74HCT240, U16 74LS138, U18 74LS00, U2 EPM7128SLC84-10, U3 LM7805_TO220, U4 AY-3-8910, U5 HM62256, U6 74HC04, U7 HM62256, U8 Z80, U9 74LS32, Y2 14.000 Mhz

Commit message: Add files via upload
Minor moves to J6/R15/16/17/18/73/J18 along with rotation and move of Q2
Parts:
- moved Q2 1.55 mm to (162.7, 143.0), turned to 0 degrees
- moved R16 1.11 mm to (32.4, 37.1)
- moved R15 1.10 mm to (30.2, 37.1)
- moved R19 1.04 mm to (34.8, 37.1)
- moved R17 1.01 mm to (37.2, 37.1)
- moved J18 1.00 mm to (42.6, 38.3)
- moved R73 1.00 mm to (46.0, 44.7)
- moved J6 0.93 mm to (35.4, 30.3)
Routing:
- net Net-(J6-Pad1): track 16.8 -> 14.6 mm
- net Net-(J6-Pad3): track 15.1 -> 16.9 mm
- net +5V: track 985.0 -> 983.4 mm
- net Net-(J7-Pin_1): track 17.2 -> 15.7 mm
- net A8: track 232.1 -> 233.4 mm
- net A14: track 343.2 -> 342.0 mm
- net ROMCS: track 152.5 -> 151.3 mm
- net VD6: track 32.7 -> 33.8 mm
- net Net-(D4-A): track 10.4 -> 9.30 mm
- net BUSAK: track 67.7 -> 68.8 mm
- net CLKAY: track 51.8 -> 50.7 mm
- net CSYNC: track 100.3 -> 101.3 mm
- net Net-(J18-Pin_2): track 114.3 -> 113.3 mm
- net Net-(J6-Pad7): track 6.21 -> 5.34 mm
- net WR: track 237.0 -> 236.2 mm
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Other:
- board text added: "ENABLE"
- board text removed: "JS_ENABLE"

Commit message: Add files via upload
Minor cosmetic changes to silkscreen and README.MD 
No changes to schematic or PCB layout.
Parts:
- moved J18 5.18 mm to (42.6, 43.5)
- moved C2 3.68 mm to (89.2, 81.5)
- moved R6 3.68 mm to (84.1, 45.5)
- moved R7 3.68 mm to (76.5, 45.5)
- moved R9 3.68 mm to (81.6, 45.5)
- moved D3 3.68 mm to (25.8, 51.1)
- moved D4 3.68 mm to (25.8, 53.7)
- moved D5 3.68 mm to (25.8, 56.2)
- moved J20 3.68 mm to (38.0, 59.3)
- moved R1 3.68 mm to (36.0, 51.1)
- moved R10 3.68 mm to (86.6, 53.1)
- moved R11 3.68 mm to (89.1, 45.5)
- moved R2 3.68 mm to (35.9, 53.7)
- moved R3 3.68 mm to (36.0, 56.2)
- moved R8 3.68 mm to (79.0, 53.1)
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Routing:
- net GND: track 931.2 -> 889.2 mm, vias 286 -> 291
- net J3-Left: track 21.4 -> 26.9 mm
- net J5-Fire3: track 44.2 -> 49.7 mm
- net CSYNC: track 101.3 -> 96.4 mm
- net NMI: track 45.9 -> 41.1 mm
- net J9-Fire2: track 24.7 -> 29.4 mm, vias 0 -> 1
- net J6-Fire: track 40.2 -> 44.4 mm
- net J1-Up: track 31.7 -> 35.8 mm
- net J2-Down: track 24.9 -> 29.0 mm
- net Net-(J6-Pad3): track 16.9 -> 20.9 mm
- net CLKAY: track 50.7 -> 46.8 mm
- net D0: track 273.5 -> 277.4 mm
- net BC1: track 57.3 -> 53.4 mm
- net Net-(J6-Pad7): track 5.34 -> 9.16 mm
- net BDIR: track 56.3 -> 52.6 mm
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Other:
- outline, holes or cut-outs redrawn
- board text added: "EEPROM 2-4/3-1 || UVEPROM 2-1/3-4 --"
- board text added: "JS ENABLE"
- board text added: "liveboxandy's Spider 48K V1.6"
- board text removed: "EEPROM 2-4/3-1 || EPROM 2-1/3-4 --"
- board text removed: "ENABLE"
