File: ZXSpider48.kicad_sch (KiCad schematic)
At the start: 123 parts, among them J1 Barrel_Jack_Switch, J11 EAR/MIC, J12 KB_CONN_05, J14 RESET, J15 ZX_48K_EDGE, J17 ON/OFF, J2 JTAG, J3 9V, J5 ROM_SW, J6 M-DIN KMDGX-9S-BS-1, J7 SPK_ON_OFF, J8 KB_CON_08, Q1 BC517, Q10 BC560, Q11 BC560, Q12 BC560, Q13 BC560, Q14 BC560, Q15 BC560, Q2 BC548, Q8 BC560, Q9 BC560, U10 27C256, U2 EPM7128SLC84-10, U3 LM7805_TO220, U5 HM62256, U6 74HC04, U7 HM62256, U8 Z80, Y2 14.000 Mhz

Commit message: Add files via upload
Corrected R58 value 470R
Added jumper for EPROM/EEPROM select
Added jumper notations
Added more buffers to clock signal
Parts:
- added J9: UV/EEPROM, Connector_PinHeader_2.54mm:PinHeader_2x02_P2.54mm_Vertical, symbol Connector_Generic:Conn_02x02_Odd_Even
- HBL1, HBR1, HTM1: footprint MountingHole:MountingHole_3.2mm_M3 -> _MOD:MountingHole_3.3mm Spectrum
- HLM1, HRM1: footprint MountingHole:MountingHole_5.3mm_M5 -> _MOD:MountingHole_5mm Spectrum
- R58: value 470K -> 470R
- U10: value 27C256 -> 27/28C256
Connections:
- net +5V: now also J9.3 (Pin_3); no longer U10.1 (VPP)
- net GND: no longer U6.1, U6.13, U6.3
- net at C20.1, R50.1: now also U6.2; no longer U6.6
- net at R50.2, Y2.1: now also U6.1; no longer U6.5
- net at D3.2 (A): now also R1.1, R15.2; no longer R15.1
- net at C20.2, R54.2: now also U6.13; no longer U6.11
- net at U6.12: now also R54.1, U6.3, Y2.2
- net at R17.1: now also J6.1; no longer D5.2 (A)
- net at R17.2, R3.1: now also D5.2 (A); no longer J6.1
- net at U6.4: now also U6.11
- net at J5.2 (Pin_2), R74.2: now also J9.2 (Pin_2); no longer U10.27 (A14)
- net at R16.1: now also J6.3; no longer D4.2 (A)
- net at R16.2, R2.1: now also D4.2 (A); no longer J6.3
- new net: U6.10, U6.5
- new net: U6.6, U6.9
- new net: J6.7, R15.1
- new net: J9.4 (Pin_4), U10.1 (VPP/A14)
- new net: J9.1 (Pin_1), U10.27 (A14/-WE)
- no-connect marks 25 -> 22
Other:
- moved on the sheet: J5, R1, R15, R16, R17, R19, R2, R3, R74, U6A, U6B, U6C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

Commit message: Add files via upload
Updated to V1,7 Added resistor for auto RGB switching. Added resistor/zener for auto AV switching. Updated README.MD
Parts:
- removed J6: M-DIN KMDGX-9S-BS-1, _MOD:KMDGX9SBS1, symbol _Symbols:KMDGX-9S-BS-1
- added D2: 12V, Diode_THT:D_DO-35_SOD27_P7.62mm_Horizontal, symbol Device:D_Zener_Small
- added J6: M-DIN KMDGX-9S-BS-1, _MOD:KMDGX9SBS1, symbol _Symbols:Mini-DIN-9
- added R20: 270R, Resistor_THT:R_Axial_DIN0204_L3.6mm_D1.6mm_P7.62mm_Horizontal, symbol Device:R
- added R21: 150R, Resistor_THT:R_Axial_DIN0207_L6.3mm_D2.5mm_P15.24mm_Horizontal, symbol Device:R
- J1: now in the parts list
- U8: MANUFACTURER_NAME Zilog -> (none); Manufacturer_Name (none) -> Zilog
Connections:
- net +12V: now also R21.2
- net +5V: now also R20.2
- net AUDIO: now also J6.8, J6.9
- net GND: now also D2.2 (A)
- net at R15.1: now also J6.7
- net at R17.1: now also J6.1
- net at R16.1: now also J6.3
- net at R19.1: now also J6.4
- new net: D2.1 (K), J6.6, R21.1
- new net: J6.2, R20.1
- no-connect marks 22 -> 21

Commit message: Tidy Up Part 2 and Release V1.8
Parts:
- Q10, Q11, Q12, Q13, Q14, Q15, Q2, Q8, Q9: footprint Package_TO_SOT_THT:TO-92_Inline -> Package_TO_SOT_THT:TO-92_Inline_Wide
- U8: MANUFACTURER_NAME (none) -> Zilog; Manufacturer_Name Zilog -> (none)
Changed lines of the file:
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@@
 	(title_block
 		(title "ZX SPIDER 48 LBA")
-		(date "2026-09-20")
-		(rev "1.7")
+		(date "2026-10-26")
+		(rev "1.8")
 		(company "Drawn By LiveBoxAndy ")
 		(comment 3 "See README.MD for more details")
@@
 			)
 		)
-		(property "Footprint" "Package_TO_SOT_THT:TO-92_Inline"
+		(property "Footprint" "Package_TO_SOT_THT:TO-92_Inline_Wide"
 			(at 299.72 230.505 0)
 			(hide yes)
@@
 			)
 		)
-		(property "Datasheet" "https://www.onsemi.com/pub/Collateral/BC550-D.pdf"
+		(property "Datasheet" ""
 			(at 294.64 228.6 0)
 			(hide yes)
@@
 			)
 		)
-		(property "Description" "0.1A Ic, 30V Vce, Small Signal NPN Transistor, TO-92"
+		(property "Description" ""
 			(at 294.64 228.6 0)
 			(hide yes)
@@
 			)
 		)
-		(property "Footprint" "Package_TO_SOT_THT:TO-92_Inline"
+		(property "Footprint" "Package_TO_SOT_THT:TO-92_Inline_Wide"
 			(at 90.805 163.83 0)
 			(hide yes)
@@
 			)
 		)
-		(property "Datasheet" "https://www.onsemi.com/pub/Collateral/BC556BTA-D.pdf"
+		(property "Datasheet" ""
 			(at 92.71 158.75 0)
 			(hide yes)
@@
 			)
 		)
-		(property "Description" "0.1A Ic, 45V Vce, PNP Small Signal Transistor, TO-92"
+		(property "Description" ""
 			(at 92.71 158.75 0)
 			(hide yes)
@@
 			)
 		)
-		(property "Footprint" "Package_TO_SOT_THT:TO-92_Inline"
+		(property "Footprint" "Package_TO_SOT_THT:TO-92_Inline_Wide"
 			(at 67.945 156.21 0)
 			(hide yes)
@@
 			)
 		)
-		(property "Datasheet" "https://www.onsemi.com/pub/Collateral/BC556BTA-D.pdf"
+		(property "Datasheet" ""
 			(at 69.85 151.13 0)
 			(hide yes)
@@
 			)
 		)
-		(property "Description" "0.1A Ic, 45V Vce, PNP Small Signal Transistor, TO-92"
+		(property "Description" ""
 			(at 69.85 151.13 0)
 			(hide yes)
@@
 			)
 		)
-		(property "Footprint" "Package_TO_SOT_THT:TO-92_Inline"
+		(property "Footprint" "Package_TO_SOT_THT:TO-92_Inline_Wide"
 			(at 56.515 173.99 0)
 			(hide yes)
@@
 			)
 		)
-		(property "Datasheet" "https://www.onsemi.com/pub/Collateral/BC556BTA-D.pdf"
+		(property "Datasheet" ""
 			(at 58.42 168.91 0)
 			(hide yes)
@@
 			)
 		)
-		(property "Description" "0.1A Ic, 45V Vce, PNP Small Signal Transistor, TO-92"
+		(property "Description" ""
 			(at 58.42 168.91 0)
 			(hide yes)
@@
 			)
 		)
-		(property "Footprint" "Package_TO_SOT_THT:TO-92_Inline"
+		(property "Footprint" "Package_TO_SOT_THT:TO-92_Inline_Wide"
 			(at 80.645 181.61 0)
 			(hide yes)
@@
 			)
 		)
-		(property "Datasheet" "https://www.onsemi.com/pub/Collateral/BC556BTA-D.pdf"
+		(property "Datasheet" ""
 			(at 82.55 176.53 0)
 			(hide yes)
@@
 			)
 		)
-		(property "Description" "0.1A Ic, 45V Vce, PNP Small Signal Transistor, TO-92"
+		(property "Description" ""
 			(at 82.55 176.53 0)
 			(hide yes)
@@
 			)
 		)
-		(property "Footprint" "Package_TO_SOT_THT:TO-92_Inline"
+		(property "Footprint" "Package_TO_SOT_THT:TO-92_Inline_Wide"
 			(at 67.945 178.054 0)
 			(hide yes)
@@
 			)
 		)
-		(property "Datasheet" "https://www.onsemi.com/pub/Collateral/BC556BTA-D.pdf"
+		(property "Datasheet" ""
 			(at 69.85 172.974 0)
 			(hide yes)
@@
 			)
 		)
-		(property "Description" "0.1A Ic, 45V Vce, PNP Small Signal Transistor, TO-92"
+		(property "Description" ""
 			(at 69.85 172.974 0)
 			(hide yes)
@@
 			)
 		)
-		(property "Footprint" "Package_TO_SOT_THT:TO-92_Inline"
+		(property "Footprint" "Package_TO_SOT_THT:TO-92_Inline_Wide"
 			(at 56.515 152.4 0)
 			(hide yes)
@@
 			)
 		)
-		(property "Datasheet" "https://www.onsemi.com/pub/Collateral/BC556BTA-D.pdf"
+		(property "Datasheet" ""
 			(at 58.42 147.32 0)
 			(hide yes)
@@
 			)
 		)
-		(property "Description" "0.1A Ic, 45V Vce, PNP Small Signal Transistor, TO-92"
+		(property "Description" ""
 			(at 58.42 147.32 0)
 			(hide yes)
@@
 			)
 		)
-		(property "Footprint" "Package_TO_SOT_THT:TO-92_Inline"
+		(property "Footprint" "Package_TO_SOT_THT:TO-92_Inline_Wide"
 			(at 79.375 160.02 0)
 			(hide yes)
@@
 			)
 		)
-		(property "Datasheet" "https://www.onsemi.com/pub/Collateral/BC556BTA-D.pdf"
+		(property "Datasheet" ""
 			(at 81.28 154.94 0)
 			(hide yes)
@@
 			)
 		)
-		(property "Description" "0.1A Ic, 45V Vce, PNP Small Signal Transistor, TO-92"
+		(property "Description" ""
 			(at 81.28 154.94 0)
 			(hide yes)
@@
 			)
 		)
-		(property "Footprint" "Package_TO_SOT_THT:TO-92_Inline"
+		(property "Footprint" "Package_TO_SOT_THT:TO-92_Inline_Wide"
 			(at 92.075 185.42 0)
 			(hide yes)
@@
 			)
 		)
-		(property "Datasheet" "https://www.onsemi.com/pub/Collateral/BC556BTA-D.pdf"
+		(property "Datasheet" ""
 			(at 93.98 180.34 0)
 			(hide yes)
@@
 			)
 		)
-		(property "Description" "0.1A Ic, 45V Vce, PNP Small Signal Transistor, TO-92"
+		(property "Description" ""
 			(at 93.98 180.34 0)
 			(hide yes)
@@
 			)
 		)
-		(property "Manufacturer_Name" "Zilog"
-			(at 345.694 106.68 0)
-			(hide yes)
-			(show_name no)
-			(do_not_autoplace no)
-			(effects
-				(font
-					(size 1.27 1.27)
-				)
-				(justify bottom)
-			)
-		)
 		(property "MF" ""
 			(at 347.472 114.808 0)
@@
 			)
 		)
-		(property "Height" ""
-			(at 332.994 103.378 0)
-			(hide yes)
-			(show_name no)
-			(do_not_autoplace no)
-			(effects
-				(font
-					(size 1.27 1.27)
-				)
-				(justify bottom)
-			)
-		)
 		(property "MP" ""
 			(at 345.44 102.362 0)
@@
 			)
 		)
-		(property "Manufacturer_Part_Number" ""
-			(at 346.456 110.49 0)
+		(property "HEIGHT" ""
+			(at 330.2 106.934 0)
+			(hide yes)
+			(show_name no)
+			(do_not_autoplace no)
+			(effects
+				(font
+					(size 1.27 1.27)
+				)
+			)
+		)
+		(property "MANUFACTURER_NAME" "Zilog"
+			(at 330.2 106.934 0)
+			(hide yes)
+			(show_name no)
+			(do_not_autoplace no)
+			(effects
+				(font
+					(size 1.27 1.27)
+				)
+			)
+		)
+		(property "MANUFACTURER_PART_NUMBER" ""
+			(at 330.2 106.934 0)
 			(hide yes)
 			(show_name no)
@@
 					(size 1.27 1.27)
 				)
-				(justify bottom)
 			)
 		)
